File: KICAD/LC_PAMV1/LC_PAM.kicad_pcb (KiCad board)
At the start: 4 copper layers, 138 x 26 mm, 25 parts, among them J1 Conn_01x04, J10 Conn_01x02, J11 Conn_01x02, J2 DC/DC, J3 Conn_01x24, J4 Conn_01x24, J5 Conn_01x02, J6 HPAB, J7 Conn_01x02_Pin, J8 Conn_01x06_Pin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

Commit message: V26-02
Routing:
- net /H5V: track 27.0 -> 25.6 mm
- net /VADD: track 22.2 -> 20.8 mm
Changed lines of the file:
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@@
 	)
 	(segment
-		(start 80.3 54.625)
-		(end 80.3 62.158)
+		(start 81.975 52.95)
+		(end 81.975 63.833)
+		(width 0.5)
+		(layer "In2.Cu")
+		(net 49)
+	)
+	(segment
+		(start 95.1664 67.5)
+		(end 95.1782 67.4882)
 		(width 0.5)
 		(layer "In2.Cu")
@@
 	)
 	(segment
-		(start 81.975 52.95)
-		(end 80.3 54.625)
+		(start 84.792 66.65)
+		(end 87.35 66.65)
 		(width 0.5)
 		(layer "In2.Cu")
@@
 	)
 	(segment
-		(start 80.3 62.158)
+		(start 81.975 63.833)
 		(end 84.792 66.65)
 		(width 0.5)
@@
 	)
 	(segment
-		(start 84.792 66.65)
-		(end 87.35 66.65)
-		(width 0.5)
-		(layer "In2.Cu")
-		(net 49)
-	)
-	(segment
-		(start 95.1664 67.5)
-		(end 95.1782 67.4882)
-		(width 0.5)
-		(layer "In2.Cu")
-		(net 49)
-	)
-	(segment
 		(start 119.359 55.299)
 		(end 120.484 56.424)
@@
 	)
 	(segment
+		(start 78.35 63.963106)
+		(end 84.752894 70.366)
+		(width 1)
+		(layer "In2.Cu")
+		(net 80)
+	)
+	(segment
+		(start 78.375 52.95)
+		(end 78.35 52.975)
+		(width 1)
+		(layer "In2.Cu")
+		(net 80)
+	)
+	(segment
 		(start 84.752894 70.366)
 		(end 85.46 70.366)
@@
 	)
 	(segment
-		(start 76.7 54.625)
-		(end 76.7 62.313106)
-		(width 1)
-		(layer "In2.Cu")
-		(net 80)
-	)
-	(segment
-		(start 78.375 52.95)
-		(end 76.7 54.625)
-		(width 1)
-		(layer "In2.Cu")
-		(net 80)
-	)
-	(segment
-		(start 76.7 62.313106)
-		(end 84.752894 70.366)
-		(width 1)
-		(layer "In2.Cu")
+		(start 78.35 52.975)
+		(end 78.35 63.963106)
+		(width 1)
+		(layer "In2.Cu")

Commit message: V23-07-25
Parts:
- added C3: 10u, Capacitor_THT:CP_Radial_D4.0mm_P1.50mm, F.Cu at (51.4, 52.6)
- added J12: Conn_01x02, Connector_PinHeader_2.54mm:PinHeader_1x02_P2.54mm_Vertical, F.Cu at (177.0, 54.4)
- added J13: Conn_01x02, Resistor_THT:R_Axial_DIN0204_L3.6mm_D1.6mm_P1.90mm_Vertical, F.Cu at (130.9, 58.1)
- added J14: Conn_01x02, Resistor_THT:R_Axial_DIN0204_L3.6mm_D1.6mm_P1.90mm_Vertical, F.Cu at (131.0, 62.1)
- added Q1: BC548, Package_TO_SOT_THT:TO-92_Inline, F.Cu at (58.9, 52.9)
- R1: value 100k -> 1k; footprint Resistor_SMD:R_0805_2012Metric_Pad1.20x1.40mm_HandSolder -> Resistor_THT:R_Axial_DIN0204_L3.6mm_D1.6mm_P2.54mm_Vertical
- moved R1 82.0 mm to (56.4, 52.7), turned to 180 degrees
- moved BT1 13.6 mm to (138.7, 64.2)
- moved J5 5.03 mm to (157.9, 71.8), turned to 180 degrees
Connections:
- net /GND renamed GND
- J1 pad 4: /V_Battery -> /V_Battery_IN
- J9 pad 1: /V_PreAmp -> /V_PreAmp_In
- R1 pad 1: /PRG -> /V_PreAmp_In
- R1 pad 2: /BAT -> Net-(Q1-B)
Routing:
- net /V_PreAmp_In: track 0.00 -> 17.5 mm
- net /BAT: track 20.9 -> 5.70 mm
- net Net-(Q1-B): track 0.00 -> 10.9 mm
- net /V_PreAmp: track 21.4 -> 13.1 mm
- net /V5: track 97.5 -> 103.9 mm
- net /V_Battery_IN: track 0.00 -> 6.25 mm
- net /V_Battery: track 140.9 -> 136.4 mm
- net /PRG: track 48.1 -> 52.0 mm
