File: KICAD/LC_PAMV1/LC_PAM.kicad_sch (KiCad schematic)
At the start: 24 parts, among them J1 Conn_01x04, J10 Conn_01x02, J11 Conn_01x02, J2 DC/DC, J3 Conn_01x24, J4 Conn_01x24, J5 Conn_01x02, J6 HPAB, J7 Conn_01x02_Pin, J8 Conn_01x06_Pin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

Commit message: v03-02-25
Parts:
- added R1: 100k, Resistor_SMD:R_0805_2012Metric_Pad1.20x1.40mm_HandSolder, symbol Device:R
- J2: footprint Connector_PinHeader_2.54mm:PinHeader_1x03_P2.54mm_Vertical -> Connector_PinHeader_2.54mm:PinHeader_1x04_P2.54mm_Vertical; symbol Connector_Generic:Conn_01x03 -> Connector_Generic:Conn_01x04
- J9: value Conn_01x03 -> Conn_01x04
Connections:
- net BAT: now also R1.2
- net GND: now also J5.1 (Pin_1)
- net PRG: now also R1.1
- net V_Battery: now also C1.1, J2.3 (Pin_3), L1.1; no longer J5.2 (Pin_2)
- removed net Vext: C1.1, J2.3 (Pin_3), J5.1 (Pin_1), L1.1
- new net nSHDN: J2.4 (Pin_4), J5.2 (Pin_2)
Other:
- moved on the sheet: J5
Changed lines of the file:
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@@
 	(wire
 		(pts
+			(xy 40.64 114.3) (xy 40.64 120.65)
+		)
+		(stroke
+			(width 0)
+			(type default)
+		)
+	)
+	(wire
+		(pts
 			(xy 247.65 69.85) (xy 265.43 69.85)
 		)
@@
 	(wire
 		(pts
+			(xy 248.92 156.21) (xy 212.09 156.21)
+		)
+		(stroke
+			(width 0)
+			(type default)
+		)
+	)
+	(wire
+		(pts
 			(xy 247.65 82.55) (xy 265.43 82.55)
 		)
@@
 	(wire
 		(pts
+			(xy 223.52 143.51) (xy 248.92 143.51)
+		)
+		(stroke
+			(width 0)
+			(type default)
+		)
+	)
+	(wire
+		(pts
 			(xy 95.25 77.47) (xy 95.25 82.55)
 		)
@@
 	(wire
 		(pts
+			(xy 248.92 143.51) (xy 248.92 148.59)
+		)
+		(stroke
+			(width 0)
+			(type default)
+		)
+	)
+	(wire
+		(pts
 			(xy 177.8 67.31) (xy 191.77 67.31)
 		)
@@
 	(wire
 		(pts
-			(xy 87.63 54.61) (xy 87.63 78.74)
+			(xy 38.1 114.3) (xy 40.64 114.3)
 		)
 		(stroke
@@
 	(wire
 		(pts
-			(xy 92.71 91.44) (xy 92.71 90.17)
+			(xy 87.63 54.61) (xy 87.63 78.74)
 		)
 		(stroke
@@
 	(wire
 		(pts
-			(xy 247.65 100.33) (xy 265.43 100.33)
+			(xy 92.71 91.44) (xy 92.71 90.17)
 		)
 		(stroke
@@
 	(wire
 		(pts
-			(xy 92.71 52.07) (xy 92.71 73.66)
+			(xy 247.65 100.33) (xy 265.43 100.33)
 		)
 		(stroke
@@
 	(wire
 		(pts
-			(xy 87.63 78.74) (xy 87.63 99.06)
+			(xy 92.71 52.07) (xy 92.71 73.66)
 		)
 		(stroke
@@
 	(wire
 		(pts
-			(xy 63.5 91.44) (xy 67.31 91.44)
+			(xy 87.63 78.74) (xy 87.63 99.06)
 		)
 		(stroke
@@
 	(wire
 		(pts
-			(xy 40.64 113.03) (xy 40.64 120.65)
+			(xy 63.5 91.44) (xy 67.31 91.44)
 		)
 		(stroke
@@
 	(wire
 		(pts
-			(xy 212.09 144.018) (xy 212.09 139.7)
+			(xy 212.09 139.7) (xy 212.09 156.21)
 		)
 		(stroke
@@
 	)
 	(label "V_Battery"
-		(at 40.64 113.03 0)
+		(at 40.64 114.3 0)
 		(fields_autoplaced yes)
 		(effects
@@
 		)
 	)
+	(label "GND"
+		(at 41.91 148.59 0)
+		(fields_autoplaced yes)
+		(effects
+			(font
+				(size 1.27 1.27)
+			)
+			(justify left bottom)
+		)
+	)
 	(label "Min"
 		(at 191.77 69.85 180)
@@
 		)
 	)
+	(label "nSHDN"
+		(at 41.91 151.13 0)
+		(fields_autoplaced yes)
+		(effects
+			(font
+				(size 1.27 1.27)
+			)
+			(justify left bottom)
+		)
+	)
 	(label "A2+"
 		(at 63.5 88.9 180)
@@
 		)
 	)
-	(label "Vext"
+	(label "V_Battery"
 		(at 91.44 140.97 0)
 		(fields_autoplaced yes)
@@
 		)
 	)
+	(label "nSHDN"
+		(at 41.91 143.51 0)
+		(fields_autoplaced yes)
+		(effects
+			(font
+				(size 1.27 1.27)
+			)
+			(justify left bottom)
+		)
+	)
 	(label "V5"
 		(at 156.21 140.97 0)
@@
 		)
 	)
-	(label "Vext"
+	(label "V_Battery"
 		(at 41.91 140.97 0)
 		(fields_autoplaced yes)
@@
 		)
 	)
-	(label "Vext"
-		(at 40.64 110.49 0)
-		(fields_autoplaced yes)
-		(effects
-			(font
-				(size 1.27 1.27)
-			)
-			(justify left bottom)
-		)
-	)
 	(label "GND"
 		(at 166.37 134.62 0)
@@
 	)
 	(symbol
-		(lib_id "Connector_Generic:Conn_01x03")
+		(lib_id "Connector_Generic:Conn_01x04")
 		(at 36.83 138.43 0)
 		(mirror y)
@@
 			)
 		)
-		(property "Footprint" "Connector_PinHeader_2.54mm:PinHeader_1x03_P2.54mm_Vertical"
+		(property "Footprint" "Connector_PinHeader_2.54mm:PinHeader_1x04_P2.54mm_Vertical"
 			(at 36.83 138.43 0)
 			(effects
@@
 			)
 		)
-		(property "Description" "Generic connector, single row, 01x03, script generated (kicad-library-utils/schlib/autogen/connector/)"
+		(property "Description" "Generic connector, single row, 01x04, script generated (kicad-library-utils/schlib/autogen/connector/)"
 			(at 36.83 138.43 0)
 			(effects
@@
 		(pin "3"
 		)
+		(pin "4"
+		)
 		(instances
 			(project ""
@@
 			)
 		)
-		(property "Value" "Conn_01x03"
+		(property "Value" "Conn_01x04"
 			(at 106.172 116.7821 0)
 			(effects
@@
 	)
 	(symbol
+		(lib_id "Device:R")
+		(at 248.92 152.4 0)
+		(unit 1)
+		(exclude_from_sim no)
+		(in_bom yes)
+		(on_board yes)
+		(dnp no)
+		(fields_autoplaced yes)
+		(property "Reference" "R1"
+			(at 250.698 151.1878 0)
+			(effects
+				(font
+					(size 1.27 1.27)
+				)
+				(justify left)
+			)
+		)
+		(property "Value" "100k"
+			(at 250.698 153.6121 0)
+			(effects
+				(font
+					(size 1.27 1.27)
+				)
+				(justify left)
+			)
+		)
+		(property "Footprint" "Resistor_SMD:R_0805_2012Metric_Pad1.20x1.40mm_HandSolder"
+			(at 247.142 152.4 90)
+			(effects
+				(font
+					(size 1.27 1.27)
+				)
+				(hide yes)
+			)
+		)
+		(property "Datasheet" "~"
+			(at 248.92 152.4 0)
+			(effects
+				(font
+					(size 1.27 1.27)
+				)
+				(hide yes)
+			)
+		)
+		(property "Description" "Resistor"
+			(at 248.92 152.4 0)
+			(effects
+				(font
+					(size 1.27 1.27)
+				)
+				(hide yes)
+			)
+		)
+		(pin "2"
+		)
+		(pin "1"
+		)
+		(instances
+			(project ""
+				(path "/20927a42-6f96-43de-a4f5-3ee83ace2c68"
+					(reference "R1")
+					(unit 1)
+				)
+			)
+		)
+	)
+	(symbol
 		(lib_id "Connector:Conn_01x07_Pin")
 		(at 36.83 76.2 0)
@@
 	(symbol
 		(lib_id "Library:Conn_01x02")
-		(at 35.56 110.49 0)
+		(at 36.83 148.59 0)
 		(mirror y)
 		(unit 1)
@@
 		(dnp no)
 		(property "Reference" "J5"
-			(at 33.528 110.5478 0)
+			(at 34.798 148.6478 0)
 			(effects
 				(font
@@
 		)
 		(property "Value" "Conn_01x02"
-			(at 33.528 112.9721 0)
+			(at 34.798 151.0721 0)
 			(effects
 				(font
@@
 		)
 		(property "Footprint" "Connector_PinHeader_2.54mm:PinHeader_1x02_P2.54mm_Vertical"
-			(at 35.56 110.49 0)
+			(at 36.83 148.59 0)
 			(effects
 				(font
@@
 		)
 		(property "Datasheet" "~"
-			(at 35.56 110.49 0)
+			(at 36.83 148.59 0)
 			(effects
 				(font
@@
 		)
 		(property "Description" "Generic connector, single row, 01x02, script generated (kicad-library-utils/schlib/autogen/connector/)"
-			(at 35.56 110.49 0)
+			(at 36.83 148.59 0)
 			(effects
 				(font

Commit message: v05-02-25
Parts:
- J9: footprint Connector_Wire:SolderWire-0.1sqmm_1x03_P3.6mm_D0.4mm_OD1mm -> Connector_Wire:SolderWire-0.1sqmm_1x04_P3.6mm_D0.4mm_OD1mm; symbol Connector_Generic:Conn_01x03 -> Connector_Generic:Conn_01x04
Connections:
- net H5V: now also J9.4 (Pin_4); no longer J9.3 (Pin_3)
- net VADD: now also J9.3 (Pin_3); no longer J9.2 (Pin_2)
- net V_Battery: now also J9.2 (Pin_2); no longer J6.4 (Pin_4), J8.1 (Pin_1), J9.1 (Pin_1)
- new net V_PreAmp: J6.4 (Pin_4), J8.1 (Pin_1), J9.1 (Pin_1)
Changed lines of the file:
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@@
-	(wire
-		(pts
-			(xy 40.64 114.3) (xy 40.64 120.65)
-		)
-		(stroke
-			(width 0)
-			(type default)
-		)
-	)
 	(wire
 		(pts
@@
 	(wire
 		(pts
-			(xy 38.1 114.3) (xy 40.64 114.3)
-		)
-		(stroke
-			(width 0)
-			(type default)
-		)
-	)
-	(wire
-		(pts
 			(xy 87.63 54.61) (xy 87.63 78.74)
 		)
@@
 		(pts
 			(xy 247.65 62.23) (xy 265.43 62.23)
+		)
+		(stroke
+			(width 0)
+			(type default)
+		)
+	)
+	(wire
+		(pts
+			(xy 97.79 118.11) (xy 99.06 118.11)
 		)
 		(stroke
@@
 	)
 	(label "H5V"
-		(at 99.06 118.11 180)
+		(at 99.06 120.65 180)
 		(fields_autoplaced yes)
 		(effects
@@
 	)
 	(label "V_Battery"
-		(at 99.06 113.03 180)
+		(at 99.06 115.57 180)
 		(fields_autoplaced yes)
 		(effects
@@
 		)
 	)
-	(label "V_Battery"
+	(label "V_PreAmp"
 		(at 41.91 46.99 0)
 		(fields_autoplaced yes)
@@
 		)
 	)
-	(label "V_Battery"
+	(label "V_PreAmp"
 		(at 41.91 76.2 0)
 		(fields_autoplaced yes)
@@
 	)
 	(label "V_Battery"
-		(at 40.64 114.3 0)
+		(at 40.64 120.65 0)
 		(fields_autoplaced yes)
 		(effects
@@
 	)
 	(label "VADD"
-		(at 99.06 115.57 180)
+		(at 97.79 118.11 180)
 		(fields_autoplaced yes)
 		(effects
@@
 			)
 			(justify left bottom)
+		)
+	)
+	(label "V_PreAmp"
+		(at 99.06 113.03 180)
+		(fields_autoplaced yes)
+		(effects
+			(font
+				(size 1.27 1.27)
+			)
+			(justify right bottom)
 		)
 	)
@@
 	)
 	(symbol
-		(lib_id "Connector_Generic:Conn_01x03")
+		(lib_id "Connector_Generic:Conn_01x04")
 		(at 104.14 115.57 0)
 		(unit 1)
@@
 		(fields_autoplaced yes)
 		(property "Reference" "J9"
-			(at 106.172 114.3578 0)
+			(at 106.172 115.6278 0)
 			(effects
 				(font
@@
 		)
 		(property "Value" "Conn_01x04"
-			(at 106.172 116.7821 0)
+			(at 106.172 118.0521 0)
 			(effects
 				(font
@@
 			)
 		)
-		(property "Footprint" "Connector_Wire:SolderWire-0.1sqmm_1x03_P3.6mm_D0.4mm_OD1mm"
+		(property "Footprint" "Connector_Wire:SolderWire-0.1sqmm_1x04_P3.6mm_D0.4mm_OD1mm"
 			(at 104.14 115.57 0)
 			(effects
@@
 			)
 		)
-		(property "Description" "Generic connector, single row, 01x03, script generated (kicad-library-utils/schlib/autogen/connector/)"
+		(property "Description" "Generic connector, single row, 01x04, script generated (kicad-library-utils/schlib/autogen/connector/)"
 			(at 104.14 115.57 0)
 			(effects
@@
 		(pin "2"
 		)
+		(pin "4"
+		)
 		(instances

Commit message: V23-07-25
Parts:
- added C3: 10u, Capacitor_THT:CP_Radial_D4.0mm_P1.50mm, symbol Device:C
- added J12: Conn_01x02, Connector_PinHeader_2.54mm:PinHeader_1x02_P2.54mm_Vertical, symbol Library:Conn_01x02
- added J13, J14: Conn_01x02, Resistor_THT:R_Axial_DIN0204_L3.6mm_D1.6mm_P1.90mm_Vertical, symbol Connector_Generic:Conn_01x02
- added Q1: BC548, Package_TO_SOT_THT:TO-92_Inline, symbol Transistor_BJT:BC548
- R1: value 100k -> 1k; footprint Resistor_SMD:R_0805_2012Metric_Pad1.20x1.40mm_HandSolder -> Resistor_THT:R_Axial_DIN0204_L3.6mm_D1.6mm_P2.54mm_Vertical
Connections:
- net BAT: no longer R1.2
- net GND: now also C3.2, J14.2 (Pin_2)
- net PRG: now also J13.2 (Pin_2), J14.1 (Pin_1); no longer R1.1
- net V5: now also J13.1 (Pin_1)
- net V_Battery: now also J12.2 (Pin_2); no longer J1.4 (Pin_4)
- net V_PreAmp: now also Q1.3 (E); no longer J9.1 (Pin_1)
- new net: C3.1, Q1.2 (B), R1.2
- new net V_Battery_IN: J1.4 (Pin_4), J12.1 (Pin_1)
- new net V_PreAmp_In: J9.1 (Pin_1), Q1.1 (C), R1.1
