File: KICAD/PreampFET_1-mare/PreampFET-mare.kicad_sch (KiCad schematic)
At the start: 18 parts, among them J1 Conn_01x02, J2 Conn_01x04, Q1 JFE2140DSGR, Q2 PMP4501V_115

Commit message: updated for fet-preamp
Connections:
- net +3V3: no longer L1.2
- new net Vcc: L1.2
Other:
- moved on the sheet: D1, J1, Q2, R7, R8, R9

Commit message: v19-12-24
Parts:
- added C4: 22uF, Capacitor_SMD:C_0603_1608Metric, symbol Device:C
- C1: value 0.1u -> 0.1uF
- C2: value 47u -> 22uF; footprint Capacitor_SMD:C_0805_2012Metric -> Capacitor_SMD:C_0603_1608Metric
- C3: value 150p -> 150pF
- R1, R3: value 10M -> 10M,1%
- R2, R4: value 1k -> 1k,0.1%
- R5, R6: value 49.9 -> 49.9,0.1%
- R7: value 360 -> 360,0.1%
- R8: value 10k -> 10k,1%
- R9: value 3.9k -> 3.9k,1%
Connections:
- net +3V3 is gone; now on net Vcc: J2.1 (Pin_1)
- net GND: now also C4.2
- net VC: now also L1.2, C4.1; no longer C1.1, C2.1, L1.1
- net Vcc: now also C1.1, C2.1, L1.1; no longer L1.2
Other:
- moved on the sheet: L1

Commit message: V23-07-25
Changed lines of the file:
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@@
 (kicad_sch
-	(version 20231120)
+	(version 20250114)
 	(generator "eeschema")
-	(generator_version "8.0")
+	(generator_version "9.0")
 	(paper "A5")
 	(title_block
@@
 	(label "B+"
 		(at 165.1 60.96 0)
-		(fields_autoplaced yes)
 		(effects
 			(font
@@
 	(label "A-"
 		(at 143.51 60.96 0)
-		(fields_autoplaced yes)
 		(effects
 			(font
@@
 	(label "B-"
 		(at 160.02 60.96 0)
-		(fields_autoplaced yes)
 		(effects
 			(font
@@
 	(label "A+"
 		(at 69.85 38.1 0)
-		(fields_autoplaced yes)
 		(effects
 			(font
@@
 	(label "S"
 		(at 109.22 78.74 0)
-		(fields_autoplaced yes)
 		(effects
 			(font
@@
 	(label "G"
 		(at 134.62 73.66 0)
-		(fields_autoplaced yes)
 		(effects
 			(font
@@
 	(label "G"
 		(at 63.5 55.88 0)
-		(fields_autoplaced yes)
 		(effects
 			(font
@@
 	(label "G"
 		(at 82.55 73.66 0)
-		(fields_autoplaced yes)
 		(effects
 			(font
@@
 	(label "B-"
 		(at 82.55 53.34 0)
-		(fields_autoplaced yes)
 		(effects
 			(font
@@
 	(label "B+"
 		(at 133.35 53.34 0)
-		(fields_autoplaced yes)
 		(effects
 			(font
@@
 	(label "A-"
 		(at 69.85 40.64 0)
-		(fields_autoplaced yes)
 		(effects
 			(font
@@
 	(label "A+"
 		(at 78.74 60.96 0)
-		(fields_autoplaced yes)
 		(effects
 			(font
@@
 	(label "S"
 		(at 63.5 96.52 0)
-		(fields_autoplaced yes)
 		(effects
 			(font
@@
 		)
 	)
+	(embedded_fonts no)
 )
