File: KICAD/PreampV5-mare/PreampV5-mare.kicad_sch (KiCad schematic)
At the start: 23 parts, among them J1 Conn_01x02, J2 Conn_01x04, U1 AD8656

Commit message: V23-07-25
Changed lines of the file:
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@@
 (kicad_sch
-	(version 20231120)
+	(version 20250114)
 	(generator "eeschema")
-	(generator_version "8.0")
+	(generator_version "9.0")
 	(paper "A5")
 	(title_block
@@
 		)
 	)
+	(embedded_fonts no)
 )
