File: KICAD/LC_PAMV4b/LC_PAMV4b.kicad_sch (KiCad schematic)
At the start: 23 parts, among them J1 Conn_01x02_Male, J2 Conn_01x02_Pin, J3 Conn_01x07_Socket, J4 DC/DC 5V, J5 Conn_01x05_Pin, J6 Conn_01x05_Pin, J7 Conn_01x03_Pin, J8 ADC_Power, J9 Conn_01x02_Pin, Q1 BC547C

Commit message: v07-10-25
Connections:
- net V_PreAmpIn: now also U1.1 (V+)
Changed lines of the file:
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@@
+		)
+	)
+	(label "V_PreAmpIn"
+		(at 130.81 50.8 180)
+		(effects
+			(font
+				(size 1.27 1.27)
+			)
+			(justify right bottom)
 		)
 	)
