File: KICAD/LC_PAMV4b/LC_PAMV4b.kicad_pcb (KiCad board)
At the start: 4 copper layers, 120 x 26 mm, 24 parts, among them J1 Conn_01x02_Male, J10 rtc, J2 Conn_01x02_Pin, J3 Conn_01x07_Socket, J4 DC/DC 5V, J5 Conn_01x05_Pin, J6 Conn_01x05_Pin, J7 Conn_01x03_Pin, J8 ADC_Power, J9 Conn_01x02_Pin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

Commit message: v07-10-25
Parts:
- A1: moved to B.Cu
- moved A1 20.4 mm to (150.1, 84.7), turned to -90 degrees
Connections:
- U1 pad 1: unconnected-(U1-V+-Pad1) -> /V_PreAmpIn
Routing:
- net /V_PreAmpIn: track 9.98 -> 29.0 mm
- net /A1: track 49.8 -> 38.3 mm
- net /SDA0: track 80.0 -> 69.2 mm
- net /EN: track 25.4 -> 36.0 mm
- net /VUSB: track 32.1 -> 41.7 mm, vias 0 -> 1
- net /HP_ON: track 63.4 -> 72.0 mm
- net /SCL0: track 83.2 -> 74.8 mm
- net /nINT: track 45.3 -> 37.2 mm
- net /V_Battery: track 149.3 -> 143.0 mm
- net /VIN_EN: track 48.8 -> 43.6 mm
- net /FSYNC: track 35.5 -> 40.8 mm
- net /IOVD: track 65.8 -> 70.8 mm
- net /BCLK: track 38.6 -> 42.9 mm
- net /SDOUT: track 34.1 -> 37.3 mm
- net /V_PreAmp: track 26.0 -> 25.1 mm
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Other:
- board text added: "LC_PAMV4b 10-05-25 05-10-25"
- board text removed: "LC_PAMV4b 10-05-25"

Commit message: V17-10-25
Parts:
- J6: value Conn_01x05_Pin -> RTC
- moved J9 1.88 mm to (196.9, 84.3)
- moved J6 0.58 mm to (200.0, 103.7)
Routing:
- net /V5: track 12.6 -> 10.5 mm
- net /VUSB: track 41.7 -> 39.9 mm
Changed lines of the file:
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@@
 	(footprint "Connector_PinHeader_2.00mm:PinHeader_1x02_P2.00mm_Vertical"
 		(layer "F.Cu")
-		(at 198.6038 83.6032 -90)
+		(at 196.8538 84.3032 -90)
 		(descr "Through hole straight pin header, 1x02, 2.00mm pitch, single row")
 		(tags "Through hole pin header THT 1x02 2.00mm single row")
@@
 	(footprint "Connector_PinHeader_2.54mm:PinHeader_1x05_P2.54mm_Vertical"
 		(layer "F.Cu")
-		(at 199.9788 103.0782 90)
+		(at 199.9788 103.6532 90)
 		(descr "Through hole straight pin header, 1x05, 2.54mm pitch, single row")
 		(tags "Through hole pin header THT 1x05 2.54mm single row")
@@
 			)
 		)
-		(property "Value" "Conn_01x05_Pin"
+		(property "Value" "RTC"
 			(at 0 12.49 90)
 			(layer "F.Fab")
@@
 		)
 		(property "Value" "Adafruit_Feather_RP2040_Adalogger"
-			(at 10.16 -45.72 -90)
+			(at 10.16 -45.72 270)
 			(layer "B.Fab")
 			(effects
@@
 	)
 	(segment
+		(start 176.2538 92.4032)
+		(end 179.2788 89.3782)
+		(width 1)
+		(layer "B.Cu")
+		(net 1)
+	)
+	(segment
+		(start 191.220674 83.8782)
+		(end 193.5038 83.8782)
+		(width 1)
+		(layer "B.Cu")
+		(net 1)
+	)
+	(segment
 		(start 176.2538 92.4282)
 		(end 176.2538 92.4032)
@@
 	)
 	(segment
-		(start 189.9828 85.116074)
-		(end 191.495674 83.6032)
+		(start 193.5038 83.8782)
+		(end 193.8038 84.1782)
 		(width 1)
 		(layer "B.Cu")
@@
 	)
 	(segment
-		(start 186.7788 89.3782)
-		(end 189.9828 86.1742)
+		(start 186.4788 89.3782)
+		(end 189.9828 85.8742)
 		(width 1)
 		(layer "B.Cu")
@@
 	)
 	(segment
-		(start 191.495674 83.6032)
-		(end 196.6038 83.6032)
+		(start 194.7288 84.1782)
+		(end 194.8538 84.3032)
 		(width 1)
 		(layer "B.Cu")
@@
 	)
 	(segment
-		(start 189.9828 86.1742)
-		(end 189.9828 85.116074)
+		(start 189.9828 85.116074)
+		(end 191.220674 83.8782)
 		(width 1)
 		(layer "B.Cu")
@@
 	)
 	(segment
-		(start 176.2538 92.4032)
-		(end 179.2788 89.3782)
+		(start 193.8038 84.1782)
+		(end 194.7288 84.1782)
 		(width 1)
 		(layer "B.Cu")
@@
 	(segment
 		(start 179.2788 89.3782)
-		(end 186.7788 89.3782)
+		(end 186.4788 89.3782)
+		(width 1)
+		(layer "B.Cu")
+		(net 1)
+	)
+	(segment
+		(start 189.9828 85.8742)
+		(end 189.9828 85.116074)
 		(width 1)
 		(layer "B.Cu")
@@
 	)
 	(segment
-		(start 201.4538 85.6532)
+		(start 201.6038 85.8032)
 		(end 213.2088 97.4082)
 		(width 1)
@@
 	)
 	(segment
-		(start 194.7048 87.0272)
-		(end 196.0788 85.6532)
-		(width 1)
-		(layer "In2.Cu")
-		(net 27)
-	)
-	(segment
 		(start 210.1788 106.8532)
 		(end 123.6038 106.8532)
@@
 	)
 	(segment
-		(start 193.1538 94.9332)
-		(end 194.7048 93.3822)
-		(width 1)
-		(layer "In2.Cu")
-		(net 27)
-	)
-	(segment
-		(start 213.2088 97.4082)
-		(end 213.2738 97.4082)
+		(start 195.9288 85.8032)
+		(end 201.6038 85.8032)
 		(width 1)
 		(layer "In2.Cu")
@@
 	)
 	(segment
+		(start 213.2088 97.4082)
+		(end 213.2738 97.4082)
+		(width 1)
+		(layer "In2.Cu")
+		(net 27)
+	)
+	(segment
 		(start 121.4038 104.6532)
 		(end 119.3038 104.6532)
@@
 	)
 	(segment
-		(start 196.0788 85.6532)
-		(end 201.4538 85.6532)
+		(start 194.7048 93.3822)
+		(end 194.7048 87.0272)
 		(width 1)
 		(layer "In2.Cu")
@@
 	)
 	(segment
-		(start 194.7048 93.3822)
-		(end 194.7048 87.0272)
+		(start 193.1538 94.9332)
+		(end 194.7048 93.3822)
 		(width 1)
 		(layer "In2.Cu")
@@
 	)
 	(segment
-		(start 193.1538 88.0032)
-		(end 195.905821 85.251179)
-		(width 1)
-		(layer "B.Cu")
-		(net 28)
-	)
-	(segment
-		(start 193.1538 89.8532)
-		(end 193.1538 88.0032)
+		(start 194.7048 87.0272)
+		(end 195.9288 85.8032)
 		(width 1)
-		(layer "B.Cu")
-		(net 28)
+		(layer "In2.Cu")
+		(net 27)
 	)
 	(segment
-		(start 196.955821 85.251179)
-		(end 198.6038 83.6032)
+		(start 193.1538 88.0032)
+		(end 196.8538 84.3032)
 		(width 1)
 		(layer "B.Cu")
@@
 	)
 	(segment
-		(start 195.905821 85.251179)
-		(end 196.955821 85.251179)
+		(start 193.1538 89.8532)
+		(end 193.1538 88.0032)
 		(width 1)
 		(layer "B.Cu")
@@
 	)
 	(segment
-		(start 199.9288 103.0282)
-		(end 197.3668 103.0282)
-		(width 1)
-		(layer "In2.Cu")
-		(net 42)
-	)
-	(segment
-		(start 199.9788 103.0782)
-		(end 199.9288 103.0282)
+		(start 199.9788 103.6532)
+		(end 199.3538 103.0282)
 		(width 1)
 		(layer "In2.Cu")
@@
 	)
 	(segment
+		(start 199.3538 103.0282)
+		(end 197.3668 103.0282)
+		(width 1)
+		(layer "In2.Cu")
+		(net 42)
+	)
+	(segment
 		(start 152.6338 84.6832)
 		(end 152.6788 84.7282)
@@
 	)
 	(segment
-		(start 199.7968 100.3782)
-		(end 196.9638 97.5452)
+		(start 205.0588 103.6082)
+		(end 201.8288 100.3782)
 		(width 0.25)
 		(layer "F.Cu")
@@
 	)
 	(segment
-		(start 205.0588 102.8832)
-		(end 202.5538 100.3782)
+		(start 201.8288 100.3782)
+		(end 199.7968 100.3782)
 		(width 0.25)
 		(layer "F.Cu")
@@
 	)
 	(segment
-		(start 205.0588 103.0782)
-		(end 205.0588 102.8832)
+		(start 199.7968 100.3782)
+		(end 196.9638 97.5452)
 		(width 0.25)
 		(layer "F.Cu")
@@
 	)
 	(segment
-		(start 202.5538 100.3782)
-		(end 199.7968 100.3782)
+		(start 205.0588 103.6532)
+		(end 205.0588 103.6082)
 		(width 0.25)
 		(layer "F.Cu")
@@
 	)
 	(segment
-		(start 207.5988 103.0632)
-		(end 203.7138 99.1782)
+		(start 207.5988 103.6532)
+		(end 207.5988 103.6482)
 		(width 0.25)
 		(layer "F.Cu")
@@
 	)
 	(segment
-		(start 196.9638 95.0052)
-		(end 195.7158 93.7572)
+		(start 207.5988 103.6482)
+		(end 203.1288 99.1782)
 		(width 0.25)
 		(layer "F.Cu")
@@
 	)
 	(segment
-		(start 207.5988 103.0782)
-		(end 207.5988 103.0632)
+		(start 203.1288 99.1782)
+		(end 201.1368 99.1782)
 		(width 0.25)
 		(layer "F.Cu")
@@
 	)
 	(segment
-		(start 187.1078 93.7572)
-		(end 178.0338 84.6832)
+		(start 196.9638 95.0052)
+		(end 195.7158 93.7572)
 		(width 0.25)
 		(layer "F.Cu")
@@
 	)
 	(segment
-		(start 203.7138 99.1782)
-		(end 201.1368 99.1782)
+		(start 187.1078 93.7572)
+		(end 178.0338 84.6832)
 		(width 0.25)
 		(layer "F.Cu")
@@
 	)
 	(segment
-		(start 197.2108 100.0852)
-		(end 196.9638 100.0852)
+		(start 202.5188 103.6432)
+		(end 200.5788 101.7032)
 		(width 0.25)
 		(layer "F.Cu")
@@
 	)
 	(segment
-		(start 198.8028 101.6772)
-		(end 197.2108 100.0852)
+		(start 200.5788 101.7032)
+		(end 198.8028 101.7032)
 		(width 0.25)
 		(layer "F.Cu")
@@
 	)
 	(segment
-		(start 202.5188 103.0782)
-		(end 202.5188 102.8432)
+		(start 202.5188 103.6532)
+		(end 202.5188 103.6432)
 		(width 0.25)
 		(layer "F.Cu")
@@
 	)
 	(segment
-		(start 201.3788 101.7032)
-		(end 198.8028 101.7032)
+		(start 198.8028 101.6772)
+		(end 197.2108 100.0852)
 		(width 0.25)
 		(layer "F.Cu")
@@
 	)
 	(segment
-		(start 202.5188 102.8432)
-		(end 201.3788 101.7032)
+		(start 197.2108 100.0852)
+		(end 196.9638 100.0852)
 		(width 0.25)
 		(layer "F.Cu")
