File: KICAD/LC_PAM4b2/LC_PAM4b2.kicad_pcb (KiCad board)
At the start: 4 copper layers, 128 x 26 mm, 22 parts, among them J1 Conn_01x02_Male, J10 Micro_SD_Board, J2 Conn_01x02_Pin, J3 Conn_01x07_Socket, J4 DC/DC 5V, J5 Conn_01x05_Pin, J6 Conn_01x05_Pin, J7 Conn_01x03_Pin, J8 ADC_Power, Q1 BC547C

Commit message: 24-12-25
Connections:
- J5 pad 5: /GND -> unconnected-(J5-Pin_5-Pad5)
Changed lines of the file:
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@@
 	(net 46 "/MISO")
 	(net 47 "/CS")
+	(net 48 "unconnected-(J5-Pin_5-Pad5)")
 	(footprint "Resistor_THT:R_Axial_DIN0204_L3.6mm_D1.6mm_P1.90mm_Vertical"
 		(layer "F.Cu")
@@
 			(layers "*.Cu" "*.Mask")
 			(remove_unused_layers no)
-			(net 9 "/GND")
+			(net 48 "unconnected-(J5-Pin_5-Pad5)")
 			(pinfunction "Pin_5")
 			(pintype "passive")

Commit message: v27-12-25
Parts:
- J6: value Conn_01x05_Pin -> RTC
- moved R4 19.6 mm to (124.1, 104.9)
- moved R5 19.5 mm to (128.1, 104.9)
- moved J8 19.4 mm to (138.5, 104.4)
- moved U1 2.42 mm to (133.4, 94.4)
Connections:
- R4 pad 1: /V_PreAmp -> /V_Battery
Routing:
- net /VIN_ADC: track 41.0 -> 24.7 mm
- net /A1: track 38.3 -> 51.0 mm
- net /EN: track 36.0 -> 28.2 mm
- net /IOVD: track 81.5 -> 88.2 mm
- net /V_PreAmp: track 25.8 -> 21.4 mm
- net /V_PreAmpIn: track 29.0 -> 33.0 mm
- net /HP_OUT: track 6.57 -> 9.00 mm
- net /VIN_EN: track 43.5 -> 45.7 mm
- net /A2+: track 7.00 -> 4.82 mm
- net /A2-: track 6.94 -> 4.82 mm
- net /SDA0: track 67.0 -> 68.0 mm
- net /SCL0: track 70.1 -> 71.1 mm
- net /SHDNZ: track 43.5 -> 44.5 mm
- net Net-(U1-VA): track 10.2 -> 9.24 mm
- net /FSYNC: track 40.8 -> 41.4 mm
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Other:
- board text added: "LC_PAMV4b2 10-05-25 05-10-25 27-12-25"
- board text removed: "LC_PAMV4b2 10-05-25 05-10-25 21-12-25"
