File: KICAD/LC_PAM4b2/LC_PAM4b2.kicad_sch (KiCad schematic)
At the start: 22 parts, among them J1 Conn_01x02_Male, J10 Micro_SD_Board, J2 Conn_01x02_Pin, J3 Conn_01x07_Socket, J4 DC/DC 5V, J5 Conn_01x05_Pin, J6 Conn_01x05_Pin, J7 Conn_01x03_Pin, J8 ADC_Power, Q1 BC547C

Commit message: 24-12-25
Parts:
- J6: value Conn_01x05_Pin -> RTC
Connections:
- net GND: no longer J5.5 (Pin_5)
Other:
- moved on the sheet: C2, H1, H2, H3, H4, J1, J10, J3, J5, J6, J7, Q1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

Commit message: v27-12-25
Connections:
- net V_Battery: now also R4.1
- net V_PreAmp: no longer R4.1
Changed lines of the file:
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@@
 		)
 	)
-	(label "V_PreAmp"
+	(label "V_Battery"
 		(at 250.19 49.53 0)
 		(effects
