File: KICAD/LC_PAMV4b1/LC_PAMV4b1.kicad_pcb (KiCad board)
At the start: 4 copper layers, 120 x 26 mm, 24 parts, among them J1 Conn_01x02_Male, J10 rtc, J2 Conn_01x02_Pin, J3 Conn_01x07_Socket, J4 DC/DC 5V, J5 Conn_01x05_Pin, J6 RTC, J7 Conn_01x03_Pin, J8 ADC_Power, J9 Conn_01x02_Pin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

Commit message: v01-02-26
Parts:
- H2, H3, H4: footprint myLibrary:MountingHole_3.2mm_M3_DIN965 -> MountingHole:MountingHole_3.2mm_M3_DIN965
- J6: value RTC -> Conn_01x05_Pin
- moved J6 0.82 mm to (199.2, 104.0)
Connections:
- R4 pad 1: /V_PreAmp -> /V_Battery
Routing:
- net /V_Battery: track 142.9 -> 165.5 mm
- net /V_PreAmp: track 25.1 -> 20.7 mm
- net /IOVD: track 71.0 -> 70.4 mm
Other:
- board text added: "LC_PAMV4b 10-05-25 05-10-25 30-01-26"
- board text removed: "LC_PAMV4b 10-05-25 05-10-25"
